File: KiCad/eobard/eobard.kicad_pcb (KiCad board)
At the start: 2 copper layers, 125.2 x 108.4 mm, 56 parts, among them J1 UART JACK LEFT, J2 RIGHT SSD1306 0.91 OLED 4pin, J3 UART Jack Right, J4 LEFT SSD1306 0.91 OLED 4pin, SW1 SW_SPST, SW10 SW_SPST, SW11 SW_SPST, SW12 SW_SPST, SW13 SW_SPST, SW14 SW_SPST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

Commit message: Updated Board Design
Parts:
- added D10: 1N4148, Diode_THT:D_DO-35_SOD27_P7.62mm_Horizontal, B.Cu at (157.0, 82.9)
- added D14: 1N4148, Diode_THT:D_DO-35_SOD27_P7.62mm_Horizontal, B.Cu at (138.0, 92.4)
- D14: moved to F.Cu
- moved J1 3.31 mm to (201.8, 121.2)
- moved J3 3.31 mm to (200.4, 123.7)
Routing:
- net UART RX: track 48.0 -> 45.9 mm
- net VCC: track 70.6 -> 72.1 mm
- net UART TX: track 55.0 -> 54.0 mm
- net (no net): vias 10 -> 9
